File: pico_ducky_pcb_v2/pico_ducky_pcb.kicad_sch (KiCad schematic)
At the start: 31 parts, among them J1 USB_A, SW1 R-667799, SW2 R-667799, U2 W25Q32JVZP, U3 RP2040, Y1 Crystal_GND24

Commit message: finish routing neopizel
Parts:
- gave numbers to parts that had none: 1
Connections:
- net RGB_DI: now also U3.40 (GPIO28_ADC2); no longer U3.15 (GPIO12)
- net USB_BOOT: no longer names the net of U3.32 (GPIO21)
Changed lines of the file:
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@@
   (no_connect (at 250.19 85.09))
   (no_connect (at 45.72 109.22))
+  (no_connect (at 250.19 118.11))
   (no_connect (at 250.19 123.19))
   (no_connect (at 250.19 125.73))
@@
   (no_connect (at 250.19 133.35))
   (no_connect (at 250.19 135.89))
-  (no_connect (at 250.19 138.43))
   (no_connect (at 250.19 140.97))
   (no_connect (at 250.19 113.03))
@@
     (stroke (width 0) (type default) (color 0 0 0 0))
   )
-  (wire (pts (xy 250.19 95.25) (xy 262.89 95.25))
-    (stroke (width 0) (type default) (color 0 0 0 0))
-  )
   (wire (pts (xy 62.23 171.45) (xy 54.61 171.45))
     (stroke (width 0) (type default) (color 0 0 0 0))
@@
     (stroke (width 0) (type default) (color 0 0 0 0))
   )
+  (wire (pts (xy 250.19 138.43) (xy 262.89 138.43))
+    (stroke (width 0) (type default) (color 0 0 0 0))
+  )
   (wire (pts (xy 205.74 43.18) (xy 200.66 43.18))
     (stroke (width 0) (type default) (color 0 0 0 0))
@@
   )
   (wire (pts (xy 200.66 43.18) (xy 198.12 43.18))
-    (stroke (width 0) (type default) (color 0 0 0 0))
-  )
-  (wire (pts (xy 250.19 118.11) (xy 262.89 118.11))
     (stroke (width 0) (type default) (color 0 0 0 0))
   )
@@
     (effects (font (size 1.27 1.27)) (justify left bottom))
   )
-  (label "RGB_DI" (at 256.54 95.25 0)
+  (label "RGB_DI" (at 254 138.43 0)
     (effects (font (size 1.27 1.27)) (justify left bottom))
   )
   (label "RGB_DI" (at 22.86 109.22 0)
-    (effects (font (size 1.27 1.27)) (justify left bottom))
-  )
-  (label "USB_BOOT" (at 252.73 118.11 0)
     (effects (font (size 1.27 1.27)) (justify left bottom))
   )
@@
   (symbol (lib_id "MIC5504:MIC5504-3.3YMT") (at 35.56 29.21 0) (unit 1)
     (in_bom yes) (on_board yes) (fields_autoplaced)
-    (property "Reference" "U?" (id 0) (at 35.56 19.05 0))
+    (property "Reference" "U1" (id 0) (at 35.56 19.05 0))
     (property "Value" "MIC5504-3.3YMT" (id 1) (at 35.56 21.59 0))
     (property "Footprint" "Package_DFN_QFN:UDFN-4-1EP_1x1mm_P0.65mm_EP0.48x0.48mm" (id 2) (at 35.56 39.37 0)
@@
       (reference "SW2") (unit 1) (value "R-667799") (footprint "R-WHATEVER:R-667799")
     )
+    (path "/3688ae9f-4d41-4c7d-bd3d-8b45a16022b7"
+      (reference "U1") (unit 1) (value "MIC5504-3.3YMT") (footprint "Package_DFN_QFN:UDFN-4-1EP_1x1mm_P0.65mm_EP0.48x0.48mm")
+    )
     (path "/5c0dfb3e-63f6-4ea6-b3ca-734edf20d662"
       (reference "U2") (unit 1) (value "W25Q32JVZP") (footprint "Package_SON:WSON-8-1EP_6x5mm_P1.27mm_EP3.4x4.3mm")
@@
       (reference "U3") (unit 1) (value "RP2040") (footprint "RP2040_minimal:RP2040-QFN-56")
     )
-    (path "/3688ae9f-4d41-4c7d-bd3d-8b45a16022b7"
-      (reference "U?") (unit 1) (value "MIC5504-3.3YMT") (footprint "Package_DFN_QFN:UDFN-4-1EP_1x1mm_P0.65mm_EP0.48x0.48mm")
-    )
     (path "/3d1c97c4-0ea6-49b5-8e16-2de5448ae48f"
