File: pcb/pico_ducky_pcb_v2/pico_ducky_pcb.kicad_pcb (KiCad board)
At the start: 4 copper layers, 14 x 30 mm, 31 parts, among them J1 USB_A, SW1 SW_SPST_GND, SW2 SW_SPST_GND, U1 MIC5504-3.3YMT, U2 W25Q32JVZP, U3 RP2040, Y1 Crystal_GND24

Commit message: WIP
Parts:
- added U4: D1213A-04V, Package_TO_SOT_SMD:SOT-563, F.Cu at (89.2, 47.9)
- J1: footprint pico-ducky-pcb-v2:USB3_A_Plug_Wuerth_629004113921_Horizontal -> Kevin_Lutzer_Lbr:USB3_A_Plug_Wuerth_629004113921_Horizontal
- SW1, SW2: value SW_SPST_GND -> R-667799; footprint pico-ducky-pcb-v2:R-667799 -> Kevin_Lutzer_Lbr:R-667799
- U1: value MIC5504-3.3YMT -> TCR2EE33; footprint Package_DFN_QFN:UDFN-4-1EP_1x1mm_P0.65mm_EP0.48x0.48mm -> Package_TO_SOT_SMD:SOT-553
- moved C6 0.20 mm to (82.3, 48.2)
- moved U1 0.20 mm to (82.3, 46.5), turned to -90 degrees
Connections:
- SW1 pad SHIELD: GND -> (no net)
- SW2 pad SHIELD: GND -> (no net)
- U1 pad 1: +3V3 -> +5V
- U1 pad 4: +5V -> +3V3
- U1 pad 5: GND -> unconnected-(U1-Pad5)
Routing:
- net +5V: track 0.00 -> 5.74 mm, vias 4 -> 3
- net /USB_+: track 7.44 -> 8.47 mm
- net GND: track 24.1 -> 24.8 mm, vias 27 -> 34
- net /USB_-: track 8.59 -> 9.11 mm, vias 0 -> 2
- net +3V3: vias 14 -> 15

Commit message: add the v3 files
Parts:
- removed JP1: SolderJumper_2_Open, Jumper:SolderJumper-2_P1.3mm_Open_RoundedPad1.0x1.5mm
- removed R1: 10k, Resistor_SMD:R_0402_1005Metric
- added Q1: 2N7002, Package_TO_SOT_SMD:SOT-23, B.Cu at (92.0, 53.0)
- added R4: 10k, Resistor_SMD:R_0402_1005Metric, F.Cu at (93.0, 53.0)
- added R8: 10k, Resistor_SMD:R_0402_1005Metric, B.Cu at (93.0, 50.1)
- added R9: NP, Resistor_SMD:R_0402_1005Metric, B.Cu at (82.0, 41.7)
- U3: footprint RP2040_minimal:RP2040-QFN-56 -> Kevin_Lutzer_Lbr:RP2040-QFN-56
- moved D1 2.27 mm to (91.2, 50.0)
- moved C12 2.00 mm to (84.8, 63.9), turned to -90 degrees
- moved C4 0.79 mm to (82.5, 58.7), turned to -90 degrees
- moved C3 0.69 mm to (91.7, 55.1), turned to -90 degrees
- moved C13 0.35 mm to (91.7, 58.7)
Connections:
- D1 pad 2: /RGB_DI -> /RGB_DI_5V
- D1 pad 3: +3V3 -> +5V
- J1 pad 5: GND -> Net-(J1-Pad5)
- SW1 pad 2: /SAFE_BOOT -> /QSPI_CS
- U3 pad 24: /SWCLK -> unconnected-(U3-Pad24)
- U3 pad 25: /SWD -> unconnected-(U3-Pad25)
- U3 pad 40: /RGB_DI -> /RGB_DI_3V3
Routing:
- net /QSPI_CS: track 13.6 -> 25.5 mm
- net Net-(J1-Pad5): track 0.00 -> 7.23 mm
- net /SAFE_BOOT: track 6.91 -> 0.00 mm
- net +5V: track 5.74 -> 11.2 mm, vias 3 -> 4
- net /RGB_DI: track 5.43 -> 0.00 mm, vias 2 -> 0
- net /RGB_DI_3V3: track 0.00 -> 5.22 mm, vias 0 -> 2
- net /RGB_DI_5V: track 0.00 -> 4.40 mm, vias 0 -> 1
- net +3V3: track 23.9 -> 20.5 mm, vias 15 -> 13
- net +1V1: track 16.0 -> 16.8 mm
- net /X_IN: track 6.20 -> 6.93 mm
- net /RESET: track 8.22 -> 8.92 mm
- net GND: track 24.8 -> 25.2 mm, vias 34 -> 27
Other:
- board text removed: "BOOT"
- board text removed: "Kevin Lutzer"
- board text removed: "RESET"
- board text removed: "RP Duck V2"
- board text removed: "SAFE"
- board text removed: "SEL"
