File: pcb/pico_ducky_pcb_v2/pico_ducky_pcb.kicad_sch (KiCad schematic)
At the start: 32 parts, among them J1 USB_A, SW1 R-667799, SW2 R-667799, U1 TCR2EE33, U2 W25Q32JVZP, U3 RP2040, U4 D1213A-04V, Y1 Crystal_GND24

Commit message: add the v3 files
Parts:
- removed JP1: SolderJumper_2_Open, Jumper:SolderJumper-2_P1.3mm_Open_RoundedPad1.0x1.5mm, symbol Jumper:SolderJumper_2_Open
- removed R1: 10k, Resistor_SMD:R_0402_1005Metric, symbol Device:R_Small
- removed U3: RP2040, RP2040_minimal:RP2040-QFN-56, symbol MCU_RaspberryPi_RP2040:RP2040
- added Q1: 2N7002, Package_TO_SOT_SMD:SOT-23, symbol Transistor_FET:2N7002
- added R4, R8: 10k, Resistor_SMD:R_0402_1005Metric, symbol Device:R_Small
- added R9: NP, Resistor_SMD:R_0402_1005Metric, symbol Device:R_Small
- added U3: RP2040, Kevin_Lutzer_Lbr:RP2040-QFN-56, symbol Kevin_Lutzer_Lbr:RP2040
Connections:
- net SAFE_BOOT is gone; now on net QSPI_CS: SW1.2 (B)
- net +1V1: now also U3.23 (DVDD), U3.45 (VREG_VOUT), U3.50 (DVDD)
- net +3V3: now also Q1.1 (G), R4.1, U3.1 (IOVDD), U3.10 (IOVDD), U3.22 (IOVDD), U3.33 (IOVDD), U3.42 (IOVDD), U3.43 (ADC_AVDD), U3.44 (VREG_IN), U3.48 (USB_VDD), U3.49 (IOVDD); no longer D1.3 (VDD)
- net +5V: now also D1.3 (VDD), R8.1
- net GND: now also R9.2, U3.19 (TESTEN), U3.57 (GND); no longer J1.5 (Shield)
- net QSPI_CS: now also U3.56 (QSPI_SS)
- net QSPI_SCLK: now also U3.52 (QSPI_SCLK)
- net QSPI_SD0: now also U3.53 (QSPI_SD0)
- net QSPI_SD1: now also U3.55 (QSPI_SD1)
- net QSPI_SD2: now also U3.54 (QSPI_SD2)
- net QSPI_SD3: now also U3.51 (QSPI_SD3)
- net RESET: now also U3.26 (RUN)
- net USBR_+: now also U3.47 (USB_DP)
- net USBR_-: now also U3.46 (USB_DM)
- net X_IN: now also U3.20 (XIN)
- net X_OUT: now also U3.21 (XOUT)
- net RGB_DI renamed RGB_DI_5V
- net RGB_DI_5V: now also Q1.3 (D), R8.2
- new net: J1.5 (Shield), R9.1
- new net RGB_DI_3V3: Q1.2 (S), R4.2, U3.40 (GPIO28_ADC2)
- no-connect marks 30 -> 32
Other:
- note added: "ESD Protection"
- note added: "Level Shifter"
- note added: "MCU"
- note added: "Regulator"
- note added: "Switches/Selectors"
- note added: "level shifter sim: https://github.com/kevinlutzer/labs/tree/main/spice/nmos-level-shifter"
- note removed: "Buttons"
- note removed: "Power"
- moved on the sheet: D1, J1, R5, SW1, SW2, U4
