File: pcb/rp_ducky.kicad_pcb (KiCad board)
At the start: 4 copper layers, 14 x 30 mm, 32 parts, among them J1 USB_A, SW1 R-667799, SW2 R-667799, U1 TCR2EE33, U2 W25Q32JVZP, U3 RP2040, U4 D1213A-04V, Y1 Crystal_GND24

Commit message: add v4 gerbers
Parts:
- removed C17: 0.1uF, Capacitor_SMD:C_0201_0603Metric
- removed R9: NP, Resistor_SMD:R_0402_1005Metric
- removed U4: D1213A-04V, Package_TO_SOT_SMD:SOT-563
- added JP1: SolderJumper_2_Open, Jumper:SolderJumper-2_P1.3mm_Open_TrianglePad1.0x1.5mm, B.Cu at (92.4, 42.2)
- added R1: 220, Resistor_SMD:R_0402_1005Metric, F.Cu at (90.8, 50.2)
- D1: value SK6812 -> LED; footprint LED_SMD:LED_SK6812_EC15_1.5x1.5mm -> LED_SMD:LED_0603_1608Metric
- moved D1 1.83 mm to (92.5, 51.0), turned to -90 degrees
Connections:
- net /RGB_DI renamed /LED
- D1 pad 1: GND -> Net-(D1-Pad1)
Routing:
- net +5V: track 5.81 -> 0.00 mm
- net +3V3: track 20.4 -> 18.7 mm, vias 13 -> 12
- net /LED: track 7.78 -> 6.20 mm, vias 1 -> 0
- net Net-(D1-Pad1): track 0.00 -> 1.29 mm
- net /USB_-: track 9.60 -> 8.59 mm, vias 2 -> 0
- net /USB_+: track 8.47 -> 7.76 mm
- net GND: track 25.8 -> 26.4 mm, vias 28 -> 26
